File: PCB/Throttle Position Sensor.kicad_pcb (KiCad board)
At the start: 2 copper layers, 45.5 x 25.8 mm, 0 parts

Commit message: Completed PCB.
Other:
- board text added: "D-JETRONIC THROTTLE POSITION SENSOR V1.0 andy@britishideas.com 2023 djetronic.org"
- board text removed: "D-JETRONIC THROTTLE POSITION SENSOR andy@britishideas.com"
Changed lines of the file:
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@@
       (outputformat 1)
       (mirror false)
-      (drillshape 1)
+      (drillshape 0)
       (scaleselection 1)
-      (outputdirectory "")
+      (outputdirectory "Manufacturing/")
     )
   )
@@
       (xy 132.202 111.609)
       (xy 129.882 111.607)
-      (xy 129.879 111.017)
-      (xy 126.362 111.017)
+      (xy 129.879 111.016)
+      (xy 127.459 111.014)
+      (xy 127.455195 109.950618)
+      (xy 127.780195 109.911618)
+      (xy 128.046 109.822)
+      (xy 128.275 109.671)
+      (xy 128.433 109.515)
+      (xy 128.545 109.36)
+      (xy 128.645 109.138)
+      (xy 128.699456 108.916424)
+      (xy 128.699 108.734)
+      (xy 128.681 108.524)
+      (xy 128.61 108.288)
+      (xy 128.488 108.067)
+      (xy 128.307 107.849)
+      (xy 128.138 107.727)
+      (xy 127.929 107.631)
+      (xy 127.757 107.582)
+      (xy 127.517 107.551)
+      (xy 127.25 107.58)
+      (xy 127.022 107.653)
+      (xy 126.834 107.751)
+      (xy 126.651 107.905)
+      (xy 126.511 108.075)
+      (xy 126.383 108.32)
+      (xy 126.322 108.52)
+      (xy 126.305 108.794)
+      (xy 126.332 109.009)
+      (xy 126.395 109.222)
+      (xy 126.508 109.423)
+      (xy 126.651 109.592)
+      (xy 126.797 109.722)
+      (xy 127.010096 109.843371)
+      (xy 127.198 109.913)
+      (xy 127.445 109.949)
+      (xy 127.442 111.014)
+      (xy 126.362 111.009)
       (xy 126.293 111.021)
       (xy 126.191 111.011)
@@
   (gr_poly
     (pts
-      (xy 167.183 91.333)
-      (xy 165.94 92.45)
-      (xy 165.84 92.55)
-      (xy 165.72 92.66)
-      (xy 165.59 92.77)
-      (xy 165.37 92.88)
-      (xy 165.22 92.93)
-      (xy 165 92.99)
-      (xy 164.81 93)
-      (xy 164.63 93)
-      (xy 164.42 92.96)
-      (xy 164.29 92.92)
-      (xy 164.13 92.86)
-      (xy 164.01 92.8)
-      (xy 163.91 92.73)
-      (xy 163.79 92.65)
-      (xy 163.62 92.48)
-      (xy 163.48 92.3)
-      (xy 163.43 92.2)
-      (xy 163.37 92.09)
-      (xy 163.33 91.98)
-      (xy 163.3 91.88)
-      (xy 163.27 91.79)
-      (xy 163.26 91.7)
-      (xy 163.25 91.64)
-      (xy 163.24 91.51)
-      (xy 163.24 91.41)
-      (xy 163.25 91.33)
-      (xy 163.25 91.24)
-      (xy 163.27 91.15)
-      (xy 163.32 90.97)
-      (xy 163.37 90.86)
-      (xy 163.43 90.74)
-      (xy 163.5 90.62)
-      (xy 163.55 90.54)
-      (xy 163.61 90.47)
-      (xy 163.69 90.38)
-      (xy 164.971 89.193)
+      (xy 166.0795 90.271)
+      (xy 165.42 90.825)
+      (xy 165.294 90.732)
+      (xy 165.151 90.649)
+      (xy 164.983 90.594)
+      (xy 164.793 90.571)
+      (xy 164.622 90.578)
+      (xy 164.4545 90.622)
+      (xy 164.293 90.697)
+      (xy 164.162 90.791)
+      (xy 164.025 90.933)
+      (xy 163.9335 91.079)
+      (xy 163.871 91.248)
+      (xy 163.8375 91.429)
+      (xy 163.837 91.582)
+      (xy 163.8695 91.758)
+      (xy 163.935 91.929)
+      (xy 164.0275 92.076)
+      (xy 164.175 92.213)
+      (xy 164.3285 92.322)
+      (xy 164.5135 92.39)
+      (xy 164.7195 92.43)
+      (xy 164.9115 92.417)
+      (xy 165.0905 92.373)
+      (xy 165.2495 92.298)
+      (xy 165.3805 92.215)
+      (xy 165.5325 92.036)
+      (xy 165.6275 91.881)
+      (xy 165.6815 91.716)
+      (xy 165.7005 91.545)
+      (xy 165.6935 91.37)
+      (xy 165.6545 91.2)
+      (xy 165.5775 91.033)
+      (xy 165.439 90.844)
+      (xy 166.0955 90.289)
+      (xy 167.1805 91.333)
+      (xy 165.9375 92.45)
+      (xy 165.8375 92.55)
+      (xy 165.7175 92.66)
+      (xy 165.5875 92.77)
+      (xy 165.3675 92.88)
+      (xy 165.2175 92.93)
+      (xy 164.9975 92.99)
+      (xy 164.8075 93)
+      (xy 164.6275 93)
+      (xy 164.4175 92.96)
+      (xy 164.2875 92.92)
+      (xy 164.1275 92.86)
+      (xy 164.0075 92.8)
+      (xy 163.9075 92.73)
+      (xy 163.7875 92.65)
+      (xy 163.6175 92.48)
+      (xy 163.4775 92.3)
+      (xy 163.4275 92.2)
+      (xy 163.3675 92.09)
+      (xy 163.3275 91.98)
+      (xy 163.2975 91.88)
+      (xy 163.2675 91.79)
+      (xy 163.2575 91.7)
+      (xy 163.2475 91.64)
+      (xy 163.2375 91.51)
+      (xy 163.2375 91.41)
+      (xy 163.2475 91.33)
+      (xy 163.2475 91.24)
+      (xy 163.2675 91.15)
+      (xy 163.3175 90.97)
+      (xy 163.3675 90.86)
+      (xy 163.4275 90.74)
+      (xy 163.4975 90.62)
+      (xy 163.5475 90.54)
+      (xy 163.6075 90.47)
+      (xy 163.6875 90.38)
+      (xy 164.9685 89.193)
     ) (layer "F.Cu") (width 0.01) (fill solid))
   (gr_poly
@@
   (gr_line (start 125.150687 110.914766) (end 125.150687 90.759129) (layer "Edge.Cuts") (width 0.014))
   (gr_line (start 146.306877 101.068869) (end 146.954528 101.133095) (layer "Edge.Cuts") (width 0.014))
-  (gr_text "D-JETRONIC\nTHROTTLE POSITION SENSOR\nandy@britishideas.com" (at 147.217 94.751) (layer "B.SilkS")
+  (gr_text "D-JETRONIC\nTHROTTLE POSITION SENSOR V1.0\nandy@britishideas.com 2023\ndjetronic.org" (at 146.994 95.589) (layer "B.SilkS")
     (effects (font (size 1.5 1.5) (thickness 0.3)) (justify mirror))
   )
